File: design.kicad_sch (KiCad schematic)
At the start: 2 parts

Commit message: Update design.kicad_sch
Other:
- note added: "1.71 V to 3.6 V"
Changed lines of the file:
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@@
     (comment 4 "<<hash>>")
+  )
+  (text "1.71 V to 3.6 V" (at 151.765 79.375 0)
+    (effects (font (size 1.27 1.27)) (justify left bottom))
   )
   (symbol (lib_id "Sensor_Motion:LIS3DH") (at 144.145 91.44 0) (unit 1)
